File: finalRoundNixie.sch (KiCad schematic (older format))
At the start: 56 parts, among them J1 Conn_01x06_Male, J2 HV_IN, J3 Conn_01x06_Female, J4 HV_OUT, Q1 MMBTA42LT1, Q10 MMBTA42LT1, Q11 AO3400, Q12 AO3400, Q13 AO3400, Q14 MMBTA42LT1, Q15 MMBTA42LT1, Q2 MMBTA42LT1, Q3 MMBTA42LT1, Q4 MMBTA42LT1, Q5 MMBTA42LT1, Q6 MMBTA42LT1, Q7 MMBTA42LT1, Q8 MMBTA42LT1, Q9 MMBTA42LT1, U1 74HC595D, U2 nixie-tube-qs27, U3 74HC595D, U4 ams1117-5.0

Commit message: changed AO3400 pin position (2 board)
Parts:
- removed Q11, Q12, Q13: AO3400, TO_SOT_Packages_SMD:SOT-23, symbol Q_NMOS_DGS
- removed U2: nixie-tube-qs27, nixie-tube-fp:qs27-1, symbol nixie-tube-qs27
- added Q11, Q12, Q13: AO3400, TO_SOT_Packages_SMD:SOT-23, symbol 2N7000
- added U?: nixie-tube, symbol nixie-tube
Connections:
- no-connect marks 1 -> 3
Changed lines of the file:
@@
 EESchema Schematic File Version 2
-LIBS:Nixie-Tube-with-shiftR-rescue
 LIBS:power
 LIBS:device
@@
 LIBS:valves
 LIBS:nixie-tube
-LIBS:Nixie-Tube-with-shiftR-cache
 EELAYER 25 0
 EELAYER END
@@
 Text Label 6025 4250 1    60   ~ 0
 Blue
-$Comp
-L Q_NMOS_DGS Q11
-U 1 1 59DF2203
-P 7925 5150
-F 0 "Q11" H 8125 5200 50  0000 L CNN
-F 1 "AO3400" H 8125 5100 50  0000 L CNN
-F 2 "TO_SOT_Packages_SMD:SOT-23" H 8125 5250 50  0001 C CNN
-F 3 "" H 7925 5150 50  0001 C CNN
-	1    7925 5150
-	1    0    0    -1
-$EndComp
-$Comp
-L Q_NMOS_DGS Q12
-U 1 1 59DF22B6
-P 8825 5175
-F 0 "Q12" H 9025 5225 50  0000 L CNN
-F 1 "AO3400" H 9025 5125 50  0000 L CNN
-F 2 "TO_SOT_Packages_SMD:SOT-23" H 9025 5275 50  0001 C CNN
-F 3 "" H 8825 5175 50  0001 C CNN
-	1    8825 5175
-	1    0    0    -1
-$EndComp
-$Comp
-L Q_NMOS_DGS Q13
-U 1 1 59DF2394
-P 9600 5175
-F 0 "Q13" H 9800 5225 50  0000 L CNN
-F 1 "AO3400" H 9800 5125 50  0000 L CNN
-F 2 "TO_SOT_Packages_SMD:SOT-23" H 9800 5275 50  0001 C CNN
-F 3 "" H 9600 5175 50  0001 C CNN
-	1    9600 5175
-	1    0    0    -1
-$EndComp
 Wire Wire Line
 	8025 5350 8025 5550
@@
 $EndComp
 $Comp
-L nixie-tube-qs27 U2
-U 1 1 5A0C1069
+L 2N7000 Q11
+U 1 1 5A0C81E8
+P 7925 5150
+F 0 "Q11" H 8125 5225 50  0000 L CNN
+F 1 "AO3400" H 8125 5150 50  0000 L CNN
+F 2 "TO_SOT_Packages_SMD:SOT-23" H 8125 5075 50  0001 L CIN
+F 3 "" H 7925 5150 50  0001 L CNN
+	1    7925 5150
+	1    0    0    -1
+$EndComp
+$Comp
+L 2N7000 Q12
+U 1 1 5A0C89DD
+P 8825 5175
+F 0 "Q12" H 9025 5250 50  0000 L CNN
+F 1 "AO3400" H 9025 5175 50  0000 L CNN
+F 2 "TO_SOT_Packages_SMD:SOT-23" H 9025 5100 50  0001 L CIN
+F 3 "" H 8825 5175 50  0001 L CNN
+	1    8825 5175
+	1    0    0    -1
+$EndComp
+$Comp
+L 2N7000 Q13
+U 1 1 5A0C8AB1
+P 9600 5175
+F 0 "Q13" H 9800 5250 50  0000 L CNN
+F 1 "AO3400" H 9800 5175 50  0000 L CNN
+F 2 "TO_SOT_Packages_SMD:SOT-23" H 9800 5100 50  0001 L CIN
+F 3 "" H 9600 5175 50  0001 L CNN
+	1    9600 5175
+	1    0    0    -1
+$EndComp
+NoConn ~ 5025 1325
+NoConn ~ 5150 1325
+$Comp
+L nixie-tube U?
+U 1 1 5A0CCC70
 P 5450 1950
-F 0 "U2" H 4875 2050 60  0000 C CNN
-F 1 "nixie-tube-qs27" H 5625 2275 60  0000 C CNN
-F 2 "nixie-tube-fp:qs27-1" H 5150 1975 60  0001 C CNN
+F 0 "U?" H 4875 2050 60  0000 C CNN
+F 1 "nixie-tube" H 5625 2275 60  0000 C CNN
+F 2 "" H 5150 1975 60  0001 C CNN
 F 3 "" H 5150 1975 60  0001 C CNN
 	1    5450 1950

Commit message: rename file according to the project
nixie-tube-display-with-shiftR is qs27 while roundxx is qs30
Parts:
- gave numbers to parts that had none: 1
Changed lines of the file:
@@
 	7325 3125 7325 3200
 $Comp
-L GND #PWR01
+L GND #PWR15
 U 1 1 59DF0537
 P 7325 3200
-F 0 "#PWR01" H 7325 2950 50  0001 C CNN
+F 0 "#PWR15" H 7325 2950 50  0001 C CNN
 F 1 "GND" H 7325 3050 50  0000 C CNN
 F 2 "" H 7325 3200 50  0001 C CNN
@@
 	6950 3775 6950 3850
 $Comp
-L GND #PWR02
+L GND #PWR14
 U 1 1 59DF0997
 P 6950 3850
-F 0 "#PWR02" H 6950 3600 50  0001 C CNN
+F 0 "#PWR14" H 6950 3600 50  0001 C CNN
 F 1 "GND" H 6950 3700 50  0000 C CNN
 F 2 "" H 6950 3850 50  0001 C CNN
@@
 	4925 5800 4925 5850
 $Comp
-L GND #PWR03
+L GND #PWR9
 U 1 1 59DEF495
 P 4925 5850
-F 0 "#PWR03" H 4925 5600 50  0001 C CNN
+F 0 "#PWR9" H 4925 5600 50  0001 C CNN
 F 1 "GND" H 4925 5700 50  0000 C CNN
 F 2 "" H 4925 5850 50  0001 C CNN
@@
 	6325 5650 6325 5725
 $Comp
-L GND #PWR04
+L GND #PWR13
 U 1 1 59DEFAF9
 P 6525 5725
-F 0 "#PWR04" H 6525 5475 50  0001 C CNN
+F 0 "#PWR13" H 6525 5475 50  0001 C CNN
 F 1 "GND" H 6525 5575 50  0000 C CNN
 F 2 "" H 6525 5725 50  0001 C CNN
@@
 $EndComp
 $Comp
-L GND #PWR05
+L GND #PWR18
 U 1 1 59DF166A
 P 8375 5950
-F 0 "#PWR05" H 8375 5700 50  0001 C CNN
+F 0 "#PWR18" H 8375 5700 50  0001 C CNN
 F 1 "GND" H 8375 5800 50  0000 C CNN
 F 2 "" H 8375 5950 50  0001 C CNN
@@
 DotU
 $Comp
-L GND #PWR06
+L GND #PWR16
 U 1 1 59E03A8E
 P 7775 2350
-F 0 "#PWR06" H 7775 2100 50  0001 C CNN
+F 0 "#PWR16" H 7775 2100 50  0001 C CNN
 F 1 "GND" H 7775 2200 50  0000 C CNN
 F 2 "" H 7775 2350 50  0001 C CNN
@@
 	5225 5925 5225 5625
 $Comp
-L GND #PWR07
+L GND #PWR4
 U 1 1 59E07C89
 P 2800 3525
-F 0 "#PWR07" H 2800 3275 50  0001 C CNN
+F 0 "#PWR4" H 2800 3275 50  0001 C CNN
 F 1 "GND" H 2800 3375 50  0000 C CNN
 F 2 "" H 2800 3525 50  0001 C CNN
@@
 	1525 5375 1700 5375
 $Comp
-L +5V #PWR08
+L +5V #PWR5
 U 1 1 59E0CEE2
 P 3000 5300
-F 0 "#PWR08" H 3000 5150 50  0001 C CNN
+F 0 "#PWR5" H 3000 5150 50  0001 C CNN
 F 1 "+5V" H 3000 5440 50  0000 C CNN
 F 2 "" H 3000 5300 50  0001 C CNN
@@
 	3000 5375 3000 5300
 $Comp
-L GND #PWR09
+L GND #PWR2
 U 1 1 59E0CFCB
 P 2200 5975
-F 0 "#PWR09" H 2200 5725 50  0001 C CNN
+F 0 "#PWR2" H 2200 5725 50  0001 C CNN
 F 1 "GND" H 2200 5825 50  0000 C CNN
 F 2 "" H 2200 5975 50  0001 C CNN
@@
 	2200 5825 2200 5975
 $Comp
-L +5V #PWR010
+L +5V #PWR6
 U 1 1 59E0E450
 P 3700 5675
-F 0 "#PWR010" H 3700 5525 50  0001 C CNN
+F 0 "#PWR6" H 3700 5525 50  0001 C CNN
 F 1 "+5V" H 3700 5815 50  0000 C CNN
 F 2 "" H 3700 5675 50  0001 C CNN
@@
 $EndComp
 $Comp
-L +5V #PWR011
+L +5V #PWR8
 U 1 1 59E0E605
 P 4700 5850
-F 0 "#PWR011" H 4700 5700 50  0001 C CNN
+F 0 "#PWR8" H 4700 5700 50  0001 C CNN
 F 1 "+5V" H 4700 5990 50  0000 C CNN
 F 2 "" H 4700 5850 50  0001 C CNN
@@
 $EndComp
 $Comp
-L +5V #PWR012
+L +5V #PWR10
 U 1 1 59E0EA7E
 P 5225 5625
-F 0 "#PWR012" H 5225 5475 50  0001 C CNN
+F 0 "#PWR10" H 5225 5475 50  0001 C CNN
 F 1 "+5V" H 5225 5765 50  0000 C CNN
 F 2 "" H 5225 5625 50  0001 C CNN
@@
 $EndComp
 $Comp
-L +5V #PWR013
+L +5V #PWR12
 U 1 1 59E0EB56
 P 6325 5725
-F 0 "#PWR013" H 6325 5575 50  0001 C CNN
+F 0 "#PWR12" H 6325 5575 50  0001 C CNN
 F 1 "+5V" H 6325 5865 50  0000 C CNN
 F 2 "" H 6325 5725 50  0001 C CNN
@@
 DotD
 $Comp
-L GND #PWR014
+L GND #PWR19
 U 1 1 59E1EE92
 P 8725 2350
-F 0 "#PWR014" H 8725 2100 50  0001 C CNN
+F 0 "#PWR19" H 8725 2100 50  0001 C CNN
 F 1 "GND" H 8725 2200 50  0000 C CNN
 F 2 "" H 8725 2350 50  0001 C CNN
@@
 	2050 3650 3325 3650
 $Comp
-L +5V #PWR015
+L +5V #PWR17
 U 1 1 59EE23C2
 P 8025 4650
-F 0 "#PWR015" H 8025 4500 50  0001 C CNN
+F 0 "#PWR17" H 8025 4500 50  0001 C CNN
 F 1 "+5V" H 8025 4790 50  0000 C CNN
 F 2 "" H 8025 4650 50  0001 C CNN
@@
 $EndComp
 $Comp
-L +5V #PWR016
+L +5V #PWR20
 U 1 1 59EE25D6
 P 8925 4675
-F 0 "#PWR016" H 8925 4525 50  0001 C CNN
+F 0 "#PWR20" H 8925 4525 50  0001 C CNN
 F 1 "+5V" H 8925 4815 50  0000 C CNN
 F 2 "" H 8925 4675 50  0001 C CNN
@@
 $EndComp
 $Comp
-L +5V #PWR017
+L +5V #PWR21
 U 1 1 59EE2686
 P 9700 4675
-F 0 "#PWR017" H 9700 4525 50  0001 C CNN
+F 0 "#PWR21" H 9700 4525 50  0001 C CNN
 F 1 "+5V" H 9700 4815 50  0000 C CNN
 F 2 "" H 9700 4675 50  0001 C CNN
@@
 STORE
 $Comp
-L +VDC #PWR018
+L +VDC #PWR3
 U 1 1 5A0A5D8C
 P 2575 3175
-F 0 "#PWR018" H 2575 3075 50  0001 C CNN
+F 0 "#PWR3" H 2575 3075 50  0001 C CNN
 F 1 "+VDC" H 2575 3425 50  0000 C CNN
 F 2 "" H 2575 3175 50  0001 C CNN
@@
 $EndComp
 $Comp
-L +VDC #PWR019
+L +VDC #PWR1
 U 1 1 5A0A64FC
 P 1525 5175
-F 0 "#PWR019" H 1525 5075 50  0001 C CNN
+F 0 "#PWR1" H 1525 5075 50  0001 C CNN
 F 1 "+VDC" H 1525 5425 50  0000 C CNN
 F 2 "" H 1525 5175 50  0001 C CNN
@@
 STORE
 $Comp
-L GND #PWR020
+L GND #PWR7
 U 1 1 5A0B1CC9
 P 4600 5675
-F 0 "#PWR020" H 4600 5425 50  0001 C CNN
+F 0 "#PWR7" H 4600 5425 50  0001 C CNN
 F 1 "GND" H 4600 5525 50  0000 C CNN
 F 2 "" H 4600 5675 50  0001 C CNN
@@
 $EndComp
 $Comp
-L GND #PWR021
+L GND #PWR11
 U 1 1 5A0B2485
 P 6225 5650
-F 0 "#PWR021" H 6225 5400 50  0001 C CNN
+F 0 "#PWR11" H 6225 5400 50  0001 C CNN
 F 1 "GND" H 6225 5500 50  0000 C CNN
 F 2 "" H 6225 5650 50  0001 C CNN
@@
 NoConn ~ 5150 1325
 $Comp
-L nixie-tube U?
+L nixie-tube U2
 U 1 1 5A0CCC70
 P 5450 1950
-F 0 "U?" H 4875 2050 60  0000 C CNN
+F 0 "U2" H 4875 2050 60  0000 C CNN
 F 1 "nixie-tube" H 5625 2275 60  0000 C CNN
 F 2 "" H 5150 1975 60  0001 C CNN

Commit message: remove silkscreen on female pins, re routed some of the tracks
Parts:
- J2: footprint Socket_Strips:Socket_Strip_Angled_1x01_Pitch2.54mm -> nixie-tube-fp:Socket_Strip_Angled_1x01_Pitch2.54mm_without_silk
- J3: footprint Socket_Strips:Socket_Strip_Angled_1x06_Pitch2.54mm -> nixie-tube-fp:Socket_Strip_Angled_1x06_Pitch2.54mm_without_silk
Changed lines of the file:
@@
 LIBS:valves
 LIBS:nixie-tube
+LIBS:finalRoundNixie-cache
 EELAYER 25 0
 EELAYER END
@@
 F 0 "J2" H 3750 1800 50  0000 C CNN
 F 1 "HV_IN" H 3750 1600 50  0000 C CNN
-F 2 "Socket_Strips:Socket_Strip_Angled_1x01_Pitch2.54mm" H 3750 1700 50  0001 C CNN
+F 2 "nixie-tube-fp:Socket_Strip_Angled_1x01_Pitch2.54mm_without_silk" H 3750 1700 50  0001 C CNN
 F 3 "" H 3750 1700 50  0001 C CNN
 	1    3750 1700
@@
 F 0 "J3" H 3525 4150 50  0000 C CNN
 F 1 "Conn_01x06_Female" H 3525 3450 50  0000 C CNN
-F 2 "Socket_Strips:Socket_Strip_Angled_1x06_Pitch2.54mm" H 3525 3850 50  0001 C CNN
+F 2 "nixie-tube-fp:Socket_Strip_Angled_1x06_Pitch2.54mm_without_silk" H 3525 3850 50  0001 C CNN
 F 3 "" H 3525 3850 50  0001 C CNN
 	1    3525 3850

Commit message: fixed various bugs
RGB led not connected properly to the mosfet
AO3400 pin orientation is not same with datasheet
move silkscreen away on neon footprint
Parts:
- removed D1: LED_CRGB, nixie-tube-fp:Rgb-Led, symbol LED_CRGB
- removed Q11, Q12, Q13: AO3400, TO_SOT_Packages_SMD:SOT-23, symbol 2N7000
- added D1: LED_RGB_BGR, nixie-tube-fp:LED_RGB_5050-6, symbol LED_RGB_BGR
- added Q11, Q12, Q13: AO3400, TO_SOT_Packages_SMD:SOT-23, symbol 2N7002
- U2: footprint (none) -> nixie-tube-fp:qs30-1
Connections:
- wire segments 66 -> 71
Other:
- moved on the sheet: R11, R12, R13
Changed lines of the file:
@@
 	7325 3125 7325 3200
 $Comp
-L GND #PWR15
+L GND #PWR01
 U 1 1 59DF0537
 P 7325 3200
-F 0 "#PWR15" H 7325 2950 50  0001 C CNN
+F 0 "#PWR01" H 7325 2950 50  0001 C CNN
 F 1 "GND" H 7325 3050 50  0000 C CNN
 F 2 "" H 7325 3200 50  0001 C CNN
@@
 	6950 3775 6950 3850
 $Comp
-L GND #PWR14
+L GND #PWR02
 U 1 1 59DF0997
 P 6950 3850
-F 0 "#PWR14" H 6950 3600 50  0001 C CNN
+F 0 "#PWR02" H 6950 3600 50  0001 C CNN
 F 1 "GND" H 6950 3700 50  0000 C CNN
 F 2 "" H 6950 3850 50  0001 C CNN
@@
 	4925 5800 4925 5850
 $Comp
-L GND #PWR9
+L GND #PWR03
 U 1 1 59DEF495
 P 4925 5850
-F 0 "#PWR9" H 4925 5600 50  0001 C CNN
+F 0 "#PWR03" H 4925 5600 50  0001 C CNN
 F 1 "GND" H 4925 5700 50  0000 C CNN
 F 2 "" H 4925 5850 50  0001 C CNN
@@
 	6325 5650 6325 5725
 $Comp
-L GND #PWR13
+L GND #PWR04
 U 1 1 59DEFAF9
 P 6525 5725
-F 0 "#PWR13" H 6525 5475 50  0001 C CNN
+F 0 "#PWR04" H 6525 5475 50  0001 C CNN
 F 1 "GND" H 6525 5575 50  0000 C CNN
 F 2 "" H 6525 5725 50  0001 C CNN
@@
 	6525 5700 6525 5725
 NoConn ~ 6325 4250
-$Comp
-L LED_CRGB D1
-U 1 1 59DF14B9
-P 8375 5750
-F 0 "D1" H 8375 6120 50  0000 C CNN
-F 1 "LED_CRGB" H 8375 5400 50  0000 C CNN
-F 2 "nixie-tube-fp:Rgb-Led" H 8375 5700 50  0001 C CNN
-F 3 "" H 8375 5700 50  0001 C CNN
-	1    8375 5750
-	0    -1   -1   0
-$EndComp
-$Comp
-L GND #PWR18
-U 1 1 59DF166A
-P 8375 5950
-F 0 "#PWR18" H 8375 5700 50  0001 C CNN
-F 1 "GND" H 8375 5800 50  0000 C CNN
-F 2 "" H 8375 5950 50  0001 C CNN
-F 3 "" H 8375 5950 50  0001 C CNN
-	1    8375 5950
-	1    0    0    -1
-$EndComp
+Text Label 8625 5175 2    60   ~ 0
+Red
+Text Label 9400 5175 2    60   ~ 0
+Green
 Text Label 7725 5150 2    60   ~ 0
-Red
-Text Label 8625 5175 2    60   ~ 0
-Green
-Text Label 9400 5175 2    60   ~ 0
 Blue
 Text Label 5825 4250 1    60   ~ 0
@@
 	8025 5350 8025 5550
 Wire Wire Line
-	8025 5550 8175 5550
+	8025 5550 9700 5550
 Wire Wire Line
 	8925 5375 8375 5375
@@
 	8375 5375 8375 5550
 Wire Wire Line
-	9700 5375 9700 5550
-Wire Wire Line
-	9700 5550 8575 5550
+	9700 5550 9700 5375
 Wire Wire Line
 	3950 1700 4625 1700
@@
 L R R11
 U 1 1 59DF3F26
-P 8025 4800
-F 0 "R11" V 8105 4800 50  0000 C CNN
-F 1 "500" V 8025 4800 50  0000 C CNN
-F 2 "Resistors_SMD:R_0603" V 7955 4800 50  0001 C CNN
-F 3 "" H 8025 4800 50  0001 C CNN
-	1    8025 4800
+P 8450 4300
+F 0 "R11" V 8530 4300 50  0000 C CNN
+F 1 "500" V 8450 4300 50  0000 C CNN
+F 2 "Resistors_SMD:R_0603" V 8380 4300 50  0001 C CNN
+F 3 "" H 8450 4300 50  0001 C CNN
+	1    8450 4300
 	1    0    0    -1
 $EndComp
@@
 L R R12
 U 1 1 59DF4051
-P 8925 4825
-F 0 "R12" V 9005 4825 50  0000 C CNN
-F 1 "500" V 8925 4825 50  0000 C CNN
-F 2 "Resistors_SMD:R_0603" V 8855 4825 50  0001 C CNN
-F 3 "" H 8925 4825 50  0001 C CNN
-	1    8925 4825
+P 8650 4300
+F 0 "R12" V 8730 4300 50  0000 C CNN
+F 1 "500" V 8650 4300 50  0000 C CNN
+F 2 "Resistors_SMD:R_0603" V 8580 4300 50  0001 C CNN
+F 3 "" H 8650 4300 50  0001 C CNN
+	1    8650 4300
 	1    0    0    -1
 $EndComp
@@
 L R R13
 U 1 1 59DF4103
-P 9700 4825
-F 0 "R13" V 9780 4825 50  0000 C CNN
-F 1 "500" V 9700 4825 50  0000 C CNN
-F 2 "Resistors_SMD:R_0603" V 9630 4825 50  0001 C CNN
-F 3 "" H 9700 4825 50  0001 C CNN
-	1    9700 4825
+P 8850 4300
+F 0 "R13" V 8930 4300 50  0000 C CNN
+F 1 "500" V 8850 4300 50  0000 C CNN
+F 2 "Resistors_SMD:R_0603" V 8780 4300 50  0001 C CNN
+F 3 "" H 8850 4300 50  0001 C CNN
+	1    8850 4300
 	1    0    0    -1
 $EndComp
@@
 DotU
 $Comp
-L GND #PWR16
+L GND #PWR05
 U 1 1 59E03A8E
 P 7775 2350
-F 0 "#PWR16" H 7775 2100 50  0001 C CNN
+F 0 "#PWR05" H 7775 2100 50  0001 C CNN
 F 1 "GND" H 7775 2200 50  0000 C CNN
 F 2 "" H 7775 2350 50  0001 C CNN
@@
 	5225 5925 5225 5625
 $Comp
-L GND #PWR4
+L GND #PWR06
 U 1 1 59E07C89
 P 2800 3525
-F 0 "#PWR4" H 2800 3275 50  0001 C CNN
+F 0 "#PWR06" H 2800 3275 50  0001 C CNN
 F 1 "GND" H 2800 3375 50  0000 C CNN
 F 2 "" H 2800 3525 50  0001 C CNN
@@
 	1525 5375 1700 5375
 $Comp
-L +5V #PWR5
+L +5V #PWR07
 U 1 1 59E0CEE2
 P 3000 5300
-F 0 "#PWR5" H 3000 5150 50  0001 C CNN
+F 0 "#PWR07" H 3000 5150 50  0001 C CNN
 F 1 "+5V" H 3000 5440 50  0000 C CNN
 F 2 "" H 3000 5300 50  0001 C CNN
@@
 	3000 5375 3000 5300
 $Comp
-L GND #PWR2
+L GND #PWR08
 U 1 1 59E0CFCB
 P 2200 5975
-F 0 "#PWR2" H 2200 5725 50  0001 C CNN
+F 0 "#PWR08" H 2200 5725 50  0001 C CNN
 F 1 "GND" H 2200 5825 50  0000 C CNN
 F 2 "" H 2200 5975 50  0001 C CNN
@@
 	2200 5825 2200 5975
 $Comp
-L +5V #PWR6
+L +5V #PWR09
 U 1 1 59E0E450
 P 3700 5675
-F 0 "#PWR6" H 3700 5525 50  0001 C CNN
+F 0 "#PWR09" H 3700 5525 50  0001 C CNN
 F 1 "+5V" H 3700 5815 50  0000 C CNN
 F 2 "" H 3700 5675 50  0001 C CNN
@@
 $EndComp
 $Comp
-L +5V #PWR8
+L +5V #PWR010
 U 1 1 59E0E605
 P 4700 5850
-F 0 "#PWR8" H 4700 5700 50  0001 C CNN
+F 0 "#PWR010" H 4700 5700 50  0001 C CNN
 F 1 "+5V" H 4700 5990 50  0000 C CNN
 F 2 "" H 4700 5850 50  0001 C CNN
@@
 $EndComp
 $Comp
-L +5V #PWR10
+L +5V #PWR011
 U 1 1 59E0EA7E
 P 5225 5625
-F 0 "#PWR10" H 5225 5475 50  0001 C CNN
+F 0 "#PWR011" H 5225 5475 50  0001 C CNN
 F 1 "+5V" H 5225 5765 50  0000 C CNN
 F 2 "" H 5225 5625 50  0001 C CNN
@@
 $EndComp
 $Comp
-L +5V #PWR12
+L +5V #PWR012
 U 1 1 59E0EB56
 P 6325 5725
-F 0 "#PWR12" H 6325 5575 50  0001 C CNN
+F 0 "#PWR012" H 6325 5575 50  0001 C CNN
 F 1 "+5V" H 6325 5865 50  0000 C CNN
 F 2 "" H 6325 5725 50  0001 C CNN
@@
 DotD
 $Comp
-L GND #PWR19
+L GND #PWR013
 U 1 1 59E1EE92
 P 8725 2350
-F 0 "#PWR19" H 8725 2100 50  0001 C CNN
+F 0 "#PWR013" H 8725 2100 50  0001 C CNN
 F 1 "GND" H 8725 2200 50  0000 C CNN
 F 2 "" H 8725 2350 50  0001 C CNN
@@
 	2050 3650 3325 3650
 $Comp
-L +5V #PWR17
+L +5V #PWR014
 U 1 1 59EE23C2
-P 8025 4650
-F 0 "#PWR17" H 8025 4500 50  0001 C CNN
-F 1 "+5V" H 8025 4790 50  0000 C CNN
-F 2 "" H 8025 4650 50  0001 C CNN
-F 3 "" H 8025 4650 50  0001 C CNN
-	1    8025 4650
-	1    0    0    -1
-$EndComp
-$Comp
-L +5V #PWR20
+P 8450 4150
+F 0 "#PWR014" H 8450 4000 50  0001 C CNN
+F 1 "+5V" H 8450 4290 50  0000 C CNN
+F 2 "" H 8450 4150 50  0001 C CNN
+F 3 "" H 8450 4150 50  0001 C CNN
+	1    8450 4150
+	1    0    0    -1
+$EndComp
+$Comp
+L +5V #PWR015
 U 1 1 59EE25D6
-P 8925 4675
-F 0 "#PWR20" H 8925 4525 50  0001 C CNN
-F 1 "+5V" H 8925 4815 50  0000 C CNN
-F 2 "" H 8925 4675 50  0001 C CNN
-F 3 "" H 8925 4675 50  0001 C CNN
-	1    8925 4675
-	1    0    0    -1
-$EndComp
-$Comp
-L +5V #PWR21
+P 8650 4150
+F 0 "#PWR015" H 8650 4000 50  0001 C CNN
+F 1 "+5V" H 8650 4290 50  0000 C CNN
+F 2 "" H 8650 4150 50  0001 C CNN
+F 3 "" H 8650 4150 50  0001 C CNN
+	1    8650 4150
+	1    0    0    -1
+$EndComp
+$Comp
+L +5V #PWR016
 U 1 1 59EE2686
-P 9700 4675
-F 0 "#PWR21" H 9700 4525 50  0001 C CNN
-F 1 "+5V" H 9700 4815 50  0000 C CNN
-F 2 "" H 9700 4675 50  0001 C CNN
-F 3 "" H 9700 4675 50  0001 C CNN
-	1    9700 4675
+P 8850 4150
+F 0 "#PWR016" H 8850 4000 50  0001 C CNN
+F 1 "+5V" H 8850 4290 50  0000 C CNN
+F 2 "" H 8850 4150 50  0001 C CNN
+F 3 "" H 8850 4150 50  0001 C CNN
+	1    8850 4150
 	1    0    0    -1
 $EndComp
@@
 STORE
 $Comp
-L +VDC #PWR3
+L +VDC #PWR017
 U 1 1 5A0A5D8C
 P 2575 3175
-F 0 "#PWR3" H 2575 3075 50  0001 C CNN
+F 0 "#PWR017" H 2575 3075 50  0001 C CNN
 F 1 "+VDC" H 2575 3425 50  0000 C CNN
 F 2 "" H 2575 3175 50  0001 C CNN
@@
 $EndComp
 $Comp
-L +VDC #PWR1
+L +VDC #PWR018
 U 1 1 5A0A64FC
 P 1525 5175
-F 0 "#PWR1" H 1525 5075 50  0001 C CNN
+F 0 "#PWR018" H 1525 5075 50  0001 C CNN
 F 1 "+VDC" H 1525 5425 50  0000 C CNN
 F 2 "" H 1525 5175 50  0001 C CNN
@@
 STORE
 $Comp
-L GND #PWR7
+L GND #PWR019
 U 1 1 5A0B1CC9
 P 4600 5675
-F 0 "#PWR7" H 4600 5425 50  0001 C CNN
+F 0 "#PWR019" H 4600 5425 50  0001 C CNN
 F 1 "GND" H 4600 5525 50  0000 C CNN
 F 2 "" H 4600 5675 50  0001 C CNN
@@
 $EndComp
 $Comp
-L GND #PWR11
+L GND #PWR020
 U 1 1 5A0B2485
 P 6225 5650
-F 0 "#PWR11" H 6225 5400 50  0001 C CNN
+F 0 "#PWR020" H 6225 5400 50  0001 C CNN
 F 1 "GND" H 6225 5500 50  0000 C CNN
 F 2 "" H 6225 5650 50  0001 C CNN
@@
 	1    0    0    -1
 $EndComp
-$Comp
-L 2N7000 Q11
-U 1 1 5A0C81E8
+NoConn ~ 5025 1325
+NoConn ~ 5150 1325
+$Comp
+L nixie-tube U2
+U 1 1 5A0CCC70
+P 5450 1950
+F 0 "U2" H 4875 2050 60  0000 C CNN
+F 1 "nixie-tube" H 5625 2275 60  0000 C CNN
+F 2 "nixie-tube-fp:qs30-1" H 5150 1975 60  0001 C CNN
+F 3 "" H 5150 1975 60  0001 C CNN
+	1    5450 1950
+	1    0    0    -1
+$EndComp
+Wire Wire Line
+	8025 4950 8450 4950
+Wire Wire Line
+	8450 4950 8450 4850
+Wire Wire Line
+	8650 4850 8650 4975
+Wire Wire Line
+	8650 4975 8925 4975
+Wire Wire Line
+	8850 4850 9700 4850
+Wire Wire Line
+	9700 4850 9700 4975
+$Comp
+L GND #PWR021
+U 1 1 5A104353
+P 8375 5550
+F 0 "#PWR021" H 8375 5300 50  0001 C CNN
+F 1 "GND" H 8375 5400 50  0000 C CNN
+F 2 "" H 8375 5550 50  0001 C CNN
+F 3 "" H 8375 5550 50  0001 C CNN
+	1    8375 5550
+	1    0    0    -1
+$EndComp
+Connection ~ 8375 5550
+$Comp
+L 2N7002 Q11
+U 1 1 5A10981C
 P 7925 5150
 F 0 "Q11" H 8125 5225 50  0000 L CNN
@@
 $EndComp
 $Comp
-L 2N7000 Q12
-U 1 1 5A0C89DD
+L 2N7002 Q12
+U 1 1 5A109F32
 P 8825 5175
 F 0 "Q12" H 9025 5250 50  0000 L CNN
@@
 $EndComp
 $Comp
-L 2N7000 Q13
-U 1 1 5A0C8AB1
+L 2N7002 Q13
+U 1 1 5A10B1D8
 P 9600 5175
 F 0 "Q13" H 9800 5250 50  0000 L CNN
@@
 	1    0    0    -1
 $EndComp
-NoConn ~ 5025 1325
-NoConn ~ 5150 1325
-$Comp
-L nixie-tube U2
-U 1 1 5A0CCC70
-P 5450 1950
-F 0 "U2" H 4875 2050 60  0000 C CNN
-F 1 "nixie-tube" H 5625 2275 60  0000 C CNN
-F 2 "" H 5150 1975 60  0001 C CNN
-F 3 "" H 5150 1975 60  0001 C CNN
-	1    5450 1950
-	1    0    0    -1
+$Comp
+L LED_RGB_BGR D1
+U 1 1 5A10E263
+P 8650 4650
+F 0 "D1" H 8650 5020 50  0000 C CNN
+F 1 "LED_RGB_BGR" H 8650 4300 50  0000 C CNN
+F 2 "nixie-tube-fp:LED_RGB_5050-6" H 8650 4600 50  0001 C CNN
+F 3 "" H 8650 4600 50  0001 C CNN
+	1    8650 4650
+	0    -1   -1   0
 $EndComp
 $EndSCHEMATC

Commit message: fixed 2 of the mmbta42 transistor pin number errors
Parts:
- removed Q14, Q15: MMBTA42LT1, TO_SOT_Packages_SMD:SOT-23, symbol Q_NPN_BCE
- added Q? (x2): MMBTA42LT1, TO_SOT_Packages_SMD:SOT-23, symbol Q_NPN_BEC
Changed lines of the file:
@@
 MOSI-OUT
-$Comp
-L Q_NPN_BCE Q14
-U 1 1 59E02747
-P 7675 2150
-F 0 "Q14" H 7875 2200 50  0000 L CNN
-F 1 "MMBTA42LT1" H 7875 2100 50  0000 L CNN
-F 2 "TO_SOT_Packages_SMD:SOT-23" H 7875 2250 50  0001 C CNN
-F 3 "" H 7675 2150 50  0001 C CNN
-	1    7675 2150
-	1    0    0    -1
-$EndComp
 $Comp
 L R R24
@@
 Connection ~ 6525 1175
 $Comp
-L Q_NPN_BCE Q15
-U 1 1 59E1EE85
-P 8625 2150
-F 0 "Q15" H 8825 2200 50  0000 L CNN
-F 1 "MMBTA42LT1" H 8825 2100 50  0000 L CNN
-F 2 "TO_SOT_Packages_SMD:SOT-23" H 8825 2250 50  0001 C CNN
-F 3 "" H 8625 2150 50  0001 C CNN
-	1    8625 2150
-	1    0    0    -1
-$EndComp
-$Comp
 L R R26
 U 1 1 59E1EE8B
@@
 	0    -1   -1   0
 $EndComp
+$Comp
+L Q_NPN_BEC Q?
+U 1 1 5A11319C
+P 7675 2150
+F 0 "Q?" H 7875 2200 50  0000 L CNN
+F 1 "MMBTA42LT1" H 7875 2100 50  0000 L CNN
+F 2 "TO_SOT_Packages_SMD:SOT-23" H 7875 2250 50  0001 C CNN
+F 3 "" H 7675 2150 50  0001 C CNN
+	1    7675 2150
+	1    0    0    -1
+$EndComp
+$Comp
+L Q_NPN_BEC Q?
+U 1 1 5A113281
+P 8625 2150
+F 0 "Q?" H 8825 2200 50  0000 L CNN
+F 1 "MMBTA42LT1" H 8825 2100 50  0000 L CNN
+F 2 "TO_SOT_Packages_SMD:SOT-23" H 8825 2250 50  0001 C CNN
+F 3 "" H 8625 2150 50  0001 C CNN
+	1    8625 2150
+	1    0    0    -1
+$EndComp
 $EndSCHEMATC
