File: NixieTube_QS30.sch (KiCad schematic (older format))
At the start: 56 parts, among them J1 Conn_01x06_Male, J2 HV_IN, J3 Conn_01x06_Female, J4 HV_OUT, Q1 MMBTA42LT1, Q10 MMBTA42LT1, Q11 AO3400, Q12 AO3400, Q13 AO3400, Q14 MMBTA42LT1, Q15 MMBTA42LT1, Q2 MMBTA42LT1, Q3 MMBTA42LT1, Q4 MMBTA42LT1, Q5 MMBTA42LT1, Q6 MMBTA42LT1, Q7 MMBTA42LT1, Q8 MMBTA42LT1, Q9 MMBTA42LT1, U1 74HC595D, U2 nixie-tube, U3 74HC595D, U4 ams1117-5.0

Commit message: checked all components, adjusted tracks
Parts:
- removed U2: nixie-tube, nixie-tube-fp:qs30-1, symbol nixie-tube
- added U?: nixie-tube-qs30, nixie-tube-fp:qs30-1, symbol nixie-tube-qs30
Changed lines of the file:
@@
 NoConn ~ 5025 1325
 NoConn ~ 5150 1325
-$Comp
-L nixie-tube U2
-U 1 1 5A0CCC70
-P 5450 1950
-F 0 "U2" H 4875 2050 60  0000 C CNN
-F 1 "nixie-tube" H 5625 2275 60  0000 C CNN
-F 2 "nixie-tube-fp:qs30-1" H 5150 1975 60  0001 C CNN
-F 3 "" H 5150 1975 60  0001 C CNN
-	1    5450 1950
-	1    0    0    -1
-$EndComp
 Wire Wire Line
 	8000 5225 8425 5225
@@
 Wire Wire Line
 	5900 2025 5900 2075
+$Comp
+L nixie-tube-qs30 U?
+U 1 1 5A159070
+P 5450 1950
+F 0 "U?" H 4875 2050 60  0000 C CNN
+F 1 "nixie-tube-qs30" H 5600 2250 60  0000 C CNN
+F 2 "nixie-tube-fp:qs30-1" H 5150 1975 60  0001 C CNN
+F 3 "" H 5150 1975 60  0001 C CNN
+	1    5450 1950
+	1    0    0    -1
+$EndComp
 $EndSCHEMATC
